File: PCB/hexapad.kicad_pcb (KiCad board)
At the start: 2 copper layers, 101 x 100 mm, 47 parts, among them J1 OLED_SCREEN, SW1 SW_Push_45deg, SW10 SW_Push_45deg, SW11 SW_Push_45deg, SW12 SW_Push_45deg, SW13 SW_Push_45deg, SW14 SW_Push_45deg, SW15 SW_Push_45deg, SW16 SW_Push_45deg, SW17 RotaryEncoder_Switch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

Commit message: finish firmware?
Parts:
- U2: moved to B.Cu
- moved U2 7.51 mm to (156.5, 32.2), turned to 180 degrees
- moved SW17 0.64 mm to (190.0, 38.6)
Routing:
- net INT: track 46.4 -> 27.0 mm
- net EC11-B: track 50.1 -> 36.9 mm, vias 1 -> 0
- net EC11-SW: track 63.9 -> 50.8 mm
- net +5V: track 114.5 -> 102.3 mm
- net EC11-A: track 47.0 -> 36.7 mm
- net GND: track 154.8 -> 146.2 mm
- net Net-(D17-DIN): track 29.2 -> 35.5 mm
- net Net-(D17-DOUT): track 13.6 -> 17.3 mm
- net SDA: track 93.2 -> 90.7 mm
- net +3V3: track 142.7 -> 141.7 mm
- net ROW1: track 106.4 -> 107.4 mm
- net SCL: track 90.4 -> 89.6 mm
- net ROW0: track 90.2 -> 90.9 mm
Other:
- board text added: "PLACE ON BACK"
